Commit message: diff_drive

File: urdf/bbot.xacro (robot description, xacro)
@@ -2,6 +2,7 @@
 <robot name="bbot" xmlns:xacro="http://www.ros.org/wiki/xacro">
 <xacro:include filename="$(find bbot_description)/urdf/materials.xacro" />
-<xacro:include filename="$(find bbot_description)/urdf/bbot.trans" />
+<!-- <xacro:include filename="$(find bbot_description)/urdf/bbot.trans" /> -->
 <xacro:include filename="$(find bbot_description)/urdf/bbot.gazebo" />
+<!-- <xacro:include filename="gazebo_control_bbot.xacro" /> -->
 <link name="base_footprint" />
 <link name="base_link">
@@ -89,5 +90,5 @@
     <origin xyz="0.0 -0.0010000000000000009 2.6077032477811457e-09" rpy="0 0 0"/>
     <mass value="0.0017100000509619655"/>
-    <inertia ixx="0.0" iyy="0.0" izz="0.0" ixy="0.0" iyz="0.0" ixz="0.0"/>
+    <inertia ixx="6.2e-07" iyy="3.7e-07" izz="3.7e-07" ixy="0.0" iyz="0.0" ixz="0.0"/>
   </inertial>
   <visual>

Commit message: lidar

File: urdf/bbot.xacro (robot description, xacro)
@@ -5,4 +5,5 @@
 <xacro:include filename="$(find bbot_description)/urdf/bbot.gazebo" />
 <!-- <xacro:include filename="gazebo_control_bbot.xacro" /> -->
+<xacro:include filename="$(find bbot_description)/urdf/lidar.xacro" />
 <link name="base_footprint" />
 <link name="base_link">
@@ -111,5 +112,5 @@
   <child link="base_link" />
 </joint>
-<joint name="baselink_lidar_joint" type="fixed">
+<joint name="laser_joint" type="fixed">
   <origin xyz="0.0 0.0 0.1875" rpy="0 0 0"/>
   <parent link="base_link"/>

Commit message: new_bbot_description

File: urdf/bbot.xacro (robot description, xacro)
@@ -2,15 +2,15 @@
 <robot name="bbot" xmlns:xacro="http://www.ros.org/wiki/xacro">
 <xacro:include filename="$(find bbot_description)/urdf/materials.xacro" />
-<!-- <xacro:include filename="$(find bbot_description)/urdf/bbot.trans" /> -->
+<xacro:include filename="$(find bbot_description)/urdf/bbot.trans" />
 <xacro:include filename="$(find bbot_description)/urdf/bbot.gazebo" />
-<!-- <xacro:include filename="gazebo_control_bbot.xacro" /> -->
-<xacro:include filename="$(find bbot_description)/urdf/lidar.xacro" />
-<xacro:include filename="$(find bbot_description)/urdf/camera.xacro" />
-<link name="base_footprint" />
+<xacro:include filename="$(find bbot_description)/urdf/camera1.xacro" />
+<xacro:include filename="$(find bbot_description)/urdf/lidar1.xacro" />
+<xacro:include filename="$(find bbot_description)/urdf/ros2_control.xacro" />
+<link name="base_footprint"></link>
 <link name="base_link">
   <inertial>
-    <origin xyz="2.1135272500541458e-15 0.0063142431636586584 0.10298851522133046" rpy="0 0 0"/>
+    <origin xyz="-0.006314243163658662 2.1121252064254716e-15 0.10298851522133046" rpy="0 0 0"/>
     <mass value="1.0491220696897063"/>
-    <inertia ixx="0.006007" iyy="0.006187" izz="0.00631" ixy="0.0" iyz="0.000632" ixz="0.0"/>
+    <inertia ixx="0.006187" iyy="0.006007" izz="0.00631" ixy="-0.0" iyz="0.0" ixz="-0.000632"/>
   </inertial>
   <visual>
@@ -32,5 +32,5 @@
     <origin xyz="0.0 0.0 0.007500000000000034" rpy="0 0 0"/>
     <mass value="0.02686061718819272"/>
-    <inertia ixx="3e-06" iyy="3e-06" izz="5e-06" ixy="-0.0" iyz="0.0" ixz="0.0"/>
+    <inertia ixx="3e-06" iyy="3e-06" izz="5e-06" ixy="0.0" iyz="0.0" ixz="-0.0"/>
   </inertial>
   <visual>
@@ -50,10 +50,10 @@
 <link name="leftwheel">
   <inertial>
-    <origin xyz="0.012499999999999997 8.195638681596229e-10 5.66244127975235e-10" rpy="0 0 0"/>
+    <origin xyz="-8.195639167318802e-10 0.012500000000000025 5.66244127975235e-10" rpy="0 0 0"/>
     <mass value="0.11821469543761903"/>
-    <inertia ixx="6.2e-05" iyy="3.7e-05" izz="3.7e-05" ixy="-0.0" iyz="0.0" ixz="-0.0"/>
+    <inertia ixx="3.7e-05" iyy="6.2e-05" izz="3.7e-05" ixy="0.0" iyz="-0.0" ixz="0.0"/>
   </inertial>
   <visual>
-    <origin xyz="-0.1125 -0.055 -0.0325" rpy="0 0 0"/>
+    <origin xyz="0.055 -0.1125 -0.0325" rpy="0 0 0"/>
     <geometry>
       <mesh filename="file://$(find bbot_description)/meshes/leftwheel_1.stl" scale="0.001 0.001 0.001"/>
@@ -62,5 +62,5 @@
   </visual>
   <collision>
-    <origin xyz="-0.1125 -0.055 -0.0325" rpy="0 0 0"/>
+    <origin xyz="0.055 -0.1125 -0.0325" rpy="0 0 0"/>
     <geometry>
       <mesh filename="file://$(find bbot_description)/meshes/leftwheel_1.stl" scale="0.001 0.001 0.001"/>
@@ -70,10 +70,10 @@
 <link name="rigthwheel">
   <inertial>
-    <origin xyz="-0.012499999999999997 8.195638681596229e-10 5.66244127975235e-10" rpy="0 0 0"/>
+    <origin xyz="-8.195638681596229e-10 -0.01250000000000008 5.66244127975235e-10" rpy="0 0 0"/>
     <mass value="0.11821469543761906"/>
-    <inertia ixx="6.2e-05" iyy="3.7e-05" izz="3.7e-05" ixy="-0.0" iyz="0.0" ixz="0.0"/>
+    <inertia ixx="3.7e-05" iyy="6.2e-05" izz="3.7e-05" ixy="0.0" iyz="0.0" ixz="0.0"/>
   </inertial>
   <visual>
-    <origin xyz="0.1125 -0.055 -0.0325" rpy="0 0 0"/>
+    <origin xyz="0.055 0.1125 -0.0325" rpy="0 0 0"/>
     <geometry>
       <mesh filename="file://$(find bbot_description)/meshes/rigthwheel_1.stl" scale="0.001 0.001 0.001"/>
@@ -82,5 +82,5 @@
   </visual>
   <collision>
-    <origin xyz="0.1125 -0.055 -0.0325" rpy="0 0 0"/>
+    <origin xyz="0.055 0.1125 -0.0325" rpy="0 0 0"/>
     <geometry>
       <mesh filename="file://$(find bbot_description)/meshes/rigthwheel_1.stl" scale="0.001 0.001 0.001"/>
@@ -90,10 +90,10 @@
 <link name="camera">
   <inertial>
-    <origin xyz="0.0 -0.0010000000000000009 2.6077032477811457e-09" rpy="0 0 0"/>
+    <origin xyz="0.0010000000000000564 2.298161660974074e-17 2.6077032477811457e-09" rpy="0 0 0"/>
     <mass value="0.0017100000509619655"/>
-    <inertia ixx="6.2e-07" iyy="3.7e-07" izz="3.7e-07" ixy="0.0" iyz="0.0" ixz="0.0"/>
+    <inertia ixx="3.7e-07" iyy="6.2e-07" izz="3.7e-07" ixy="-0.0" iyz="0.0" ixz="0.0"/>
   </inertial>
   <visual>
-    <origin xyz="-0.0 0.1025 -0.175" rpy="0 0 0"/>
+    <origin xyz="-0.1025 -0.0 -0.175" rpy="0 0 0"/>
     <geometry>
       <mesh filename="file://$(find bbot_description)/meshes/camera_1.stl" scale="0.001 0.001 0.001"/>
@@ -102,5 +102,5 @@
   </visual>
   <collision>
-    <origin xyz="-0.0 0.1025 -0.175" rpy="0 0 0"/>
+    <origin xyz="-0.1025 -0.0 -0.175" rpy="0 0 0"/>
     <geometry>
       <mesh filename="file://$(find bbot_description)/meshes/camera_1.stl" scale="0.001 0.001 0.001"/>
@@ -108,28 +108,28 @@
   </collision>
 </link>
-<joint name="basefootprint_baselink_joint" type="fixed">
-  <origin xyz="0 0 0" rpy="0 0 0" />
-  <parent link="base_footprint" />
-  <child link="base_link" />
+<joint name="footprint_base_joint" type="fixed">
+  <origin xyz="0.0 0.0 0.0" rpy="0 0 0"/>
+  <parent link="base_footprint"/>
+  <child link="base_link"/>
 </joint>
-<joint name="laser_joint" type="fixed">
+<joint name="base_lidar_joint" type="fixed">
   <origin xyz="0.0 0.0 0.1875" rpy="0 0 0"/>
   <parent link="base_link"/>
   <child link="lidar"/>
 </joint>
-<joint name="baselink_leftwheel_joint" type="continuous">
-  <origin xyz="0.1125 0.055 0.0325" rpy="0 0 0"/>
+<joint name="base_leftwheel_joint" type="continuous">
+  <origin xyz="-0.055 0.1125 0.0325" rpy="0 0 0"/>
   <parent link="base_link"/>
   <child link="leftwheel"/>
-  <axis xyz="-1.0 0.0 0.0"/>
+  <axis xyz="0.0 -1.0 0.0"/>
 </joint>
-<joint name="baselink_rightwheel_joint" type="continuous">
-  <origin xyz="-0.1125 0.055 0.0325" rpy="0 0 0"/>
+<joint name="base_rightwheel_joint" type="continuous">
+  <origin xyz="-0.055 -0.1125 0.0325" rpy="0 0 0"/>
   <parent link="base_link"/>
   <child link="rigthwheel"/>
-  <axis xyz="-1.0 0.0 0.0"/>
+  <axis xyz="0.0 -1.0 0.0"/>
 </joint>
-<joint name="baselink_camera_joint" type="fixed">
-  <origin xyz="0.0 -0.1025 0.175" rpy="0 0 0"/>
+<joint name="base_camera_joint" type="fixed">
+  <origin xyz="0.1025 0.0 0.175" rpy="0 0 0"/>
   <parent link="base_link"/>
   <child link="camera"/>

File: urdf/camera1.xacro (robot description, xacro)
@@ -1,4 +1,5 @@
 <?xml version="1.0"?>
 <robot xmlns:xacro="http://www.ros.org/wiki/xacro" >
+    <link name="camera_link_optical"></link>
     <joint name="camera_optical_joint" type="fixed">
         <parent link="camera"/>
@@ -6,7 +7,6 @@
         <origin xyz="0 0 0" rpy="${-pi/2} 0 ${-pi/2}"/>
     </joint>
-    <link name="camera_link_optical"></link>
     <gazebo reference="camera">
-        <material>Gazebo/Red</material>
+        <!-- <material>Gazebo/Red</material> -->
         <sensor name="camera" type="camera">
             <pose> 0 0 0 0 0 0 </pose>
